File: GWR-pcb/daughterboard.kicad_sch (KiCad schematic)
At the start: 2 parts, among them SW2 SW_SPST, SW3 SW_SPST

Commit message: update to use GPIO expander, minor fixes
Parts:
- removed SW2: SW_SPST, Button_Switch_THT:SW_Tactile_SPST_Angled_PTS645Vx83-2LFS, symbol Switch:SW_SPST
- removed SW3: SW_SPST, Button_Switch_SMD:SW_SPST_EVQQ2, symbol Switch:SW_SPST
Other:
- note removed: "angled switch"
Changed lines of the file:
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@@
 	(generator_version "10.0")
 	(paper "A4")
-	(text "angled switch"
-		(exclude_from_sim no)
-		(at 64.262 41.91 0)
-		(effects
-			(font
-				(size 1.27 1.27)
-			)
-		)
-	)
-	(symbol
-		(lib_id "Switch:SW_SPST")
-		(at 64.77 50.8 0)
-		(unit 1)
-		(body_style 1)
-		(exclude_from_sim no)
-		(in_bom yes)
-		(on_board yes)
-		(in_pos_files yes)
-		(dnp no)
-		(fields_autoplaced yes)
-		(property "Reference" "SW2"
-			(at 64.77 44.45 0)
-			(show_name no)
-			(do_not_autoplace no)
-			(effects
-				(font
-					(size 1.27 1.27)
-				)
-			)
-		)
-		(property "Value" "SW_SPST"
-			(at 64.77 46.99 0)
-			(show_name no)
-			(do_not_autoplace no)
-			(effects
-				(font
-					(size 1.27 1.27)
-				)
-			)
-		)
-		(property "Footprint" "Button_Switch_THT:SW_Tactile_SPST_Angled_PTS645Vx83-2LFS"
-			(at 64.77 50.8 0)
-			(hide yes)
-			(show_name no)
-			(do_not_autoplace no)
-			(effects
-				(font
-					(size 1.27 1.27)
-				)
-			)
-		)
-		(property "Datasheet" "https://www.littelfuse.com/assetdocs/littelfuse-c-k-tactile-pts645v-series-datasheet?assetguid=5014fb06-c6ac-482c-8b16-1ea09e49f7c0"
-			(at 64.77 50.8 0)
-			(hide yes)
-			(show_name no)
-			(do_not_autoplace no)
-			(effects
-				(font
-					(size 1.27 1.27)
-				)
-			)
-		)
-		(property "Description" "Single Pole Single Throw (SPST) switch"
-			(at 64.77 50.8 0)
-			(hide yes)
-			(show_name no)
-			(do_not_autoplace no)
-			(effects
-				(font
-					(size 1.27 1.27)
-				)
-			)
-		)
-		(pin "1"
-		)
-		(pin "2"
-		)
-		(instances
-			(project "GWR-pcb"
-				(path "/5ba9b62f-22ef-4dbd-b34f-1e4d5ec66edc"
-					(reference "SW2")
-					(unit 1)
-				)
-			)
-		)
-	)
-	(symbol
-		(lib_id "Switch:SW_SPST")
-		(at 100.33 69.85 0)
-		(unit 1)
-		(body_style 1)
-		(exclude_from_sim no)
-		(in_bom yes)
-		(on_board yes)
-		(in_pos_files yes)
-		(dnp no)
-		(fields_autoplaced yes)
-		(property "Reference" "SW3"
-			(at 100.33 63.5 0)
-			(show_name no)
-			(do_not_autoplace no)
-			(effects
-				(font
-					(size 1.27 1.27)
-				)
-			)
-		)
-		(property "Value" "SW_SPST"
-			(at 100.33 66.04 0)
-			(show_name no)
-			(do_not_autoplace no)
-			(effects
-				(font
-					(size 1.27 1.27)
-				)
-			)
-		)
-		(property "Footprint" "Button_Switch_SMD:SW_SPST_EVQQ2"
-			(at 100.33 69.85 0)
-			(hide yes)
-			(show_name no)
-			(do_not_autoplace no)
-			(effects
-				(font
-					(size 1.27 1.27)
-				)
-			)
-		)
-		(property "Datasheet" ""
-			(at 100.33 69.85 0)
-			(hide yes)
-			(show_name no)
-			(do_not_autoplace no)
-			(effects
-				(font
-					(size 1.27 1.27)
-				)
-			)
-		)
-		(property "Description" "Single Pole Single Throw (SPST) switch"
-			(at 100.33 69.85 0)
-			(hide yes)
-			(show_name no)
-			(do_not_autoplace no)
-			(effects
-				(font
-					(size 1.27 1.27)
-				)
-			)
-		)
-		(pin "1"
-		)
-		(pin "2"
-		)
-		(instances
-			(project "GWR-pcb"
-				(path "/5ba9b62f-22ef-4dbd-b34f-1e4d5ec66edc"
-					(reference "SW3")
-					(unit 1)
-				)
-			)
-		)
-	)
 	(sheet_instances
 		(path "/"

Commit message: minor fixes
Parts:
- added J10, J11, J12, J5, J6, J7, J8, J9: Conn_01x02, Connector_PinHeader_1.27mm:PinHeader_1x02_P1.27mm_Vertical, symbol Connector_Generic:Conn_01x02
- added J3: Conn_01x02, Connector_Wire:SolderWire-0.15sqmm_1x02_P4mm_D0.5mm_OD1.5mm, symbol Connector_Generic:Conn_01x02
- added J4: Conn_01x12, Connector_FFC-FPC:Hirose_FH12-12S-0.5SH_1x12-1MP_P0.50mm_Horizontal, symbol Connector_Generic:Conn_01x12
- added TP12: RES, TestPoint:TestPoint_Pad_D1.0mm, symbol Connector:TestPoint
Connections:
- new net BUTTON_A: J4.12 (Pin_12), J5.1 (Pin_1)
- new net BUTTON_B: J4.11 (Pin_11), J6.1 (Pin_1)
- new net BUTTON_C: J4.10 (Pin_10), J7.1 (Pin_1)
- new net BUTTON_D: J4.9 (Pin_9), J8.1 (Pin_1)
- new net BUTTON_E: J4.8 (Pin_8), J9.1 (Pin_1)
- new net BUTTON_F: J10.1 (Pin_1), J4.7 (Pin_7)
- new net BUTTON_G: J11.1 (Pin_1), J4.6 (Pin_6)
- new net BUTTON_H: J12.1 (Pin_1), J4.5 (Pin_5)
- new net GND_DAUGHTER: J10.2 (Pin_2), J11.2 (Pin_2), J12.2 (Pin_2), J4.1 (Pin_1), J5.2 (Pin_2), J6.2 (Pin_2), J7.2 (Pin_2), J8.2 (Pin_2), J9.2 (Pin_2)
- new net MOTOR_HIGH: J3.2 (Pin_2), J4.2 (Pin_2)
- new net MOTOR_LOW: J3.1 (Pin_1), J4.3 (Pin_3)
- new net SIG_RESERVED1: J4.4 (Pin_4), TP12.1
Other:
- note added: "FFC type: B"
- note added: "NOTICE: FFC connector flipped vertically for proper alignment"
