File: GWR-pcb/GWR-pcb.kicad_pcb (KiCad board)
At the start: 2 copper layers, 92.5 x 39 mm, 65 parts, among them J1 Conn_01x11, J10 Conn_01x02, J11 Conn_01x02, J12 Conn_01x02, J2 Conn_01x12, J3 Conn_01x02, J4 Conn_01x12, J5 Conn_01x02, J6 Conn_01x02, J7 Conn_01x02, J8 Conn_01x02, J9 Conn_01x02, Q1 AO3400A, SW1 SW_DIP_x01, SW2 Angled_Mode, SW3 Angled_RST, U1 AMS1117-1.5, U2 XIAO-ESP32-S3-Plus-SMD, U3 MAX98357A, U4 74AUP1G32, U5 MCP23S17x-x-SS, U6 ADXL343

Commit message: pcb layout changes
Parts:
- added REF**: Mousebites OSHPARK Panel, glibri:Mousebites OSHPARK Panel, F.Cu at (99.0, 52.0)
- added REF**: Mousebites OSHPARK Panel, glibri:Mousebites OSHPARK Panel, F.Cu at (124.2, 46.9)
- TP12: value GND -> RES
Connections:
- J10 pad 2: GND -> GND_DAUGHTER
- J11 pad 2: GND -> GND_DAUGHTER
- J12 pad 2: GND -> GND_DAUGHTER
- J4 pad 1: GND -> GND_DAUGHTER
- J5 pad 2: GND -> GND_DAUGHTER
- J6 pad 2: GND -> GND_DAUGHTER
- J7 pad 2: GND -> GND_DAUGHTER
- J8 pad 2: GND -> GND_DAUGHTER
- J9 pad 2: GND -> GND_DAUGHTER
Routing:
- net GND: track 70.4 -> 74.9 mm, vias 82 -> 85
- net /AUDIO_-: track 16.6 -> 15.3 mm, vias 2 -> 1
- net /AUDIO_+: track 15.7 -> 14.5 mm, vias 2 -> 1
Other:
- board size 92.5 x 39 mm -> 99.3 x 39 mm
- rule pad_to_mask_clearance: 0.1 -> 0.0508
- board text added: "TongueTyper"
- board text removed: "GW:R"

Commit message: release A
Parts:
- added C10: TBD, Capacitor_SMD:C_0603_1608Metric, F.Cu at (110.5, 51.4)
- moved J10 0.71 mm to (103.2, 50.4)
- moved J11 0.71 mm to (117.2, 54.4)
- moved J12 0.71 mm to (119.2, 50.4)
- moved J3 0.71 mm to (113.2, 57.4)
- moved J4 0.71 mm to (111.2, 43.4)
- moved J5 0.71 mm to (108.2, 54.4)
- moved J6 0.71 mm to (106.2, 50.4)
- moved J7 0.71 mm to (114.2, 54.4)
- moved J8 0.71 mm to (116.2, 50.4)
- moved J9 0.71 mm to (105.2, 54.4)
- moved REF** 0.71 mm to (103.9, 34.2)
- moved REF** 0.71 mm to (108.7, 59.2)
- moved REF** 0.71 mm to (123.5, 46.9)
- moved REF** 0.71 mm to (108.7, 37.2)
- moved REF** 0.71 mm to (105.4, 65.2)
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Routing:
- net GND: vias 85 -> 95
Other:
- board size 99.3 x 39 mm -> 98.6 x 39 mm
