File: GWR-pcb/GWR-pcb.kicad_sch (KiCad schematic)
At the start: 47 parts, among them J1 Conn_01x11, J2 Conn_01x12, M1 Motor_DC, Q1 AO3400A, SW1 SW_DIP_x01, SW2 Angled_Mode, SW3 Angled_RST, U1 AMS1117-1.5, U2 XIAO-ESP32-S3-Plus-SMD, U3 MAX98357A, U4 74AUP1G32, U5 MCP23S17x-x-SS, U6 ADXL343

Commit message: pcb layout changes
Other:
- note added: "Gain: create fake trace connecting to Vdd for 6 dB (lowest) gain"
- note added: "watch out for high current draw regulator limited to 700 mA shared with all 3v3 devices"
- moved on the sheet: C3, C5, JP1

Commit message: release A
Parts:
- added C10: TBD, Capacitor_SMD:C_0603_1608Metric, symbol Device:C
Connections:
- net MOTOR_HIGH: now also C10.1
- net MOTOR_LOW: now also C10.2
Other:
- moved on the sheet: D1
Changed lines of the file:
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@@
 	)
 	(junction
+		(at 111.76 201.93)
+		(diameter 0)
+		(color 0 0 0 0)
+	)
+	(junction
 		(at 46.99 193.04)
 		(diameter 0)
@@
 	)
 	(junction
+		(at 111.76 182.88)
+		(diameter 0)
+		(color 0 0 0 0)
+	)
+	(junction
 		(at 309.88 191.77)
 		(diameter 0)
@@
 	(wire
 		(pts
+			(xy 111.76 182.88) (xy 121.92 182.88)
+		)
+		(stroke
+			(width 0)
+			(type default)
+		)
+	)
+	(wire
+		(pts
 			(xy 212.09 125.73) (xy 213.36 125.73)
 		)
@@
 	(wire
 		(pts
-			(xy 86.36 201.93) (xy 104.14 201.93)
+			(xy 86.36 201.93) (xy 111.76 201.93)
+		)
+		(stroke
+			(width 0)
+			(type default)
+		)
+	)
+	(wire
+		(pts
+			(xy 111.76 182.88) (xy 111.76 190.5)
 		)
 		(stroke
@@
 	(wire
 		(pts
+			(xy 111.76 201.93) (xy 121.92 201.93)
+		)
+		(stroke
+			(width 0)
+			(type default)
+		)
+	)
+	(wire
+		(pts
 			(xy 340.36 77.47) (xy 341.63 77.47)
 		)
@@
 	(wire
 		(pts
+			(xy 111.76 198.12) (xy 111.76 201.93)
+		)
+		(stroke
+			(width 0)
+			(type default)
+		)
+	)
+	(wire
+		(pts
 			(xy 148.59 185.42) (xy 191.77 185.42)
 		)
@@
 	(wire
 		(pts
-			(xy 86.36 182.88) (xy 104.14 182.88)
+			(xy 86.36 182.88) (xy 111.76 182.88)
 		)
 		(stroke
@@
 	(wire
 		(pts
-			(xy 104.14 182.88) (xy 104.14 190.5)
+			(xy 121.92 182.88) (xy 121.92 190.5)
 		)
 		(stroke
@@
 	(wire
 		(pts
-			(xy 104.14 198.12) (xy 104.14 201.93)
+			(xy 121.92 198.12) (xy 121.92 201.93)
 		)
 		(stroke
@@
 	(symbol
 		(lib_id "Device:C")
+		(at 111.76 194.31 0)
+		(unit 1)
+		(body_style 1)
+		(exclude_from_sim no)
+		(in_bom yes)
+		(on_board yes)
+		(in_pos_files yes)
+		(dnp no)
+		(property "Reference" "C10"
+			(at 115.316 192.786 0)
+			(show_name no)
+			(do_not_autoplace no)
+			(effects
+				(font
+					(size 1.27 1.27)
+				)
+				(justify left)
+			)
+		)
+		(property "Value" "TBD"
+			(at 115.316 195.326 0)
+			(show_name no)
+			(do_not_autoplace no)
+			(effects
+				(font
+					(size 1.27 1.27)
+				)
+				(justify left)
+			)
+		)
+		(property "Footprint" "Capacitor_SMD:C_0603_1608Metric"
+			(at 112.7252 198.12 0)
+			(hide yes)
+			(show_name no)
+			(do_not_autoplace no)
+			(effects
+				(font
+					(size 1.27 1.27)
+				)
+			)
+		)
+		(property "Datasheet" ""
+			(at 111.76 194.31 0)
+			(hide yes)
+			(show_name no)
+			(do_not_autoplace no)
+			(effects
+				(font
+					(size 1.27 1.27)
+				)
+			)
+		)
+		(property "Description" "Unpolarized capacitor"
+			(at 111.76 194.31 0)
+			(hide yes)
+			(show_name no)
+			(do_not_autoplace no)
+			(effects
+				(font
+					(size 1.27 1.27)
+				)
+			)
+		)
+		(pin "1"
+		)
+		(pin "2"
+		)
+		(instances
+			(project "GWR-pcb"
+				(path "/45165c3b-8e6b-4141-b243-555b44fd49a6"
+					(reference "C10")
+					(unit 1)
+				)
+			)
+		)
+	)
+	(symbol
+		(lib_id "Device:C")
 		(at 59.69 186.69 0)
 		(unit 1)
@@
 	(symbol
 		(lib_id "PCM_Diode_AKL:S1A")
-		(at 104.14 194.31 90)
+		(at 121.92 194.31 90)
 		(unit 1)
 		(body_style 1)
@@
 		(fields_autoplaced yes)
 		(property "Reference" "D1"
-			(at 106.68 193.0399 90)
+			(at 124.46 193.0399 90)
 			(show_name no)
 			(do_not_autoplace no)
@@
 		)
 		(property "Value" "S1A"
-			(at 106.68 195.5799 90)
+			(at 124.46 195.5799 90)
 			(show_name no)
 			(do_not_autoplace no)
@@
 		)
 		(property "Footprint" "PCM_Diode_SMD_AKL:D_SMA"
-			(at 104.14 194.31 0)
+			(at 121.92 194.31 0)
 			(hide yes)
 			(show_name no)
@@
 		)
 		(property "Datasheet" "https://www.tme.eu/Document/f79bd540b2075b703f85044ae73d5af4/s1ab-s1mb.pdf"
-			(at 104.14 194.31 0)
+			(at 121.92 194.31 0)
 			(hide yes)
 			(show_name no)
@@
 		)
 		(property "Description" "SMA Diode, Rectifier, 50V, 1A, Alternate KiCad Library"
-			(at 104.14 194.31 0)
+			(at 121.92 194.31 0)
 			(hide yes)
 			(show_name no)
