File: PCB/Rev A/GWR-pcb/GWR-pcb.kicad_sch (KiCad schematic)
At the start: 48 parts, among them J1 Conn_01x11, J2 Conn_01x12, M1 Motor_DC, Q1 AO3400A, SW1 SW_DIP_x01, SW2 Angled_Mode, SW3 Angled_RST, U1 AMS1117-1.5, U2 XIAO-ESP32-S3-Plus-SMD, U3 MAX98357A, U4 74AUP1G32, U5 MCP23S17x-x-SS, U6 ADXL343

Commit message: shuffle PCB files around as we prep for next revision
Other:
- note removed: "SPI ctrl byte 0 1 0 0 A2 A1 A0 RW (0100000X) can disable and just use CS with HAEN bit =0"
Changed lines of the file:
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@@
-		)
-	)
-	(text "SPI ctrl byte\n0 1 0 0 A2 A1 A0 RW\n(0100000X)\ncan disable and just use CS with HAEN bit =0"
-		(exclude_from_sim no)
-		(at 240.03 67.056 0)
-		(effects
-			(font
-				(size 1.27 1.27)
-			)
 		)
 	)
